File: MultiPurposeNode/hardware/MysensorsShield/MysensorsShield.kicad_sch (KiCad schematic)
At the start: 20 parts, among them J1 TEMP SENSOR, J2 IR RECEIVER, J3 RADIO1, J4 RADIO2, J5 STEMMA, Q1 2N3904, U1 NRF24L01_Breakout

Commit message: MultiPurposeNode Rev.1 shield complete
Parts:
- D2: value RX LED -> RX
- D3: value TX LED -> TX
- D4: value ERR LED -> ERR
Changed lines of the file:
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@@
       (effects (font (size 1.27 1.27)) (justify right))
     )
-    (property "Value" "RX LED" (at 96.52 37.1475 90)
+    (property "Value" "RX" (at 96.52 37.1475 90)
       (effects (font (size 1.27 1.27)) (justify right))
     )
@@
       (effects (font (size 1.27 1.27)) (justify right))
     )
-    (property "Value" "TX LED" (at 109.22 37.1475 90)
+    (property "Value" "TX" (at 109.22 37.1475 90)
       (effects (font (size 1.27 1.27)) (justify right))
     )
@@
       (effects (font (size 1.27 1.27)) (justify right))
     )
-    (property "Value" "ERR LED" (at 121.92 37.1475 90)
-      (effects (font (size 1.27 1.27)) (justify right))
-    )
+    (property "Value" "ERR" (at 121.92 37.1475 90)
+      (effects (font (size 1.27 1.27)) (justify right))
+    )
